File: esp32_wroom_wearable.sch (EAGLE design)
At the start: 15 parts, among them J2 TYPE-C-31-M-12, U1 ESP32-S3-WROOM-1-N16R2, U5 USBLC6-2SC6

Commit message: Completed design files
Parts:
- added C10, C11, C7: 100nF, OPL_Capacitor:CERAMIC-100NF-25V-10%-X7R(0402)
- added C12, C13, C20, C5, C6, C8: 0.1uF, SparkFun-Capacitors:0.1UF-0402-16V-10%
- added C14, C15: 10uF, OPL_Capacitor:CERAMIC-10UF-6.3V-20%-X5R(0402)
- added C18, C19: 4.7uF, OPL_Capacitor:CERAMIC-4.7UF-6.3V-20%-X5R(0402)
- added C9: 1.0uF, SparkFun-Capacitors:1.0UF-0402-16V-10%
- added D1: 20V-1A, OPL_Discrete_Semiconductor:SMD-DIODE-SCHOTTKY-20V-1A(SOD-123)
- added D2: BLUE-0402, OPL_Optoelectronics:SMD-LED-CLEAR-BLUE(0402)
- added IC1: BMI055, BMI055:BMI055
- added J1: CORTEX_DEBUG_SMD, SparkFun-Connectors:CORTEX_DEBUG_SMD
- added J3: (no value), SparkFun-Connectors:QWIIC_CONNECTORJS-1MM
- added J4: TYPE-C-31-M-12, TYPE-C-31-M-12:TYPE-C-31-M-12
- added J5: (no value), SparkFun-Connectors:JST_2MM_MALE
- added M1: MOTOR10MM, SparkFun-Electromechanical:MOTOR10MM
- added MK1: ICS-41350, ICS-41350:ICS-41350
- added Q1: 2.5A/30V/105mΩ, SparkFun-DiscreteSemi:MOSFET_PCH-DMG2307L
- added R2: 10M, SparkFun-Resistors:RESISTOR0402
- added R3, R4: 4.7K, SparkFun-Resistors:RESISTOR0402
- added R5: 5.1k, SparkFun-Resistors:5.6KOHM-0603-1/10W-1%
- added R7: 2K, SparkFun-Resistors:RESISTOR0402
- added R8: 470, SparkFun-Resistors:RESISTOR0402
- added SW1: PCM12SMTR, PCM12SMTR:PCM12SMTR
- added U2: DRV2605LDGSR, DRV2605LDGSR:DRV2605LDGSR
- added U3: BME688, BME688:BME688
- added U4: MIC5504-3.3YM5_TR, MIC5504-3.3YM5_TR:MIC5504-3.3YM5_TR
- added U6: USBLC6-2SC6, USBLC6-2SC6:USBLC6-2SC6
- added Y1: FC-135_32.7680KA-A0, FC-135_32.7680KA-A0:FC-135_32.7680KA-A0
- C2: value 22uF -> 8pF; device 04026D226MAT2A:04026D226MAT2A -> SparkFun-Capacitors:6PF-0402-50V-0.5%
- C3: value 0.1uF -> 8pF; device SparkFun-Capacitors:0.1UF-0402-16V-10% -> SparkFun-Capacitors:6PF-0402-50V-0.5%
- C4: value 0.1uF -> 22uF; device SparkFun-Capacitors:0.1UF-0402-16V-10% -> 04026D226MAT2A:04026D226MAT2A
- J2: value TYPE-C-31-M-12 -> 53261-0471; device TYPE-C-31-M-12:TYPE-C-31-M-12 -> 53261-0471:53261-0471
- R9: value 5.1k -> 10K; device SparkFun-Resistors:5.6KOHM-0603-1/10W-1% -> SparkFun-Resistors:RESISTOR0402
- U5: value USBLC6-2SC6 -> MCP73831T-2ATI/OT; device USBLC6-2SC6:USBLC6-2SC6 -> MCP73831T-2ATI_OT:MCP73831T-2ATI/OT
- renumbered C25 to C16, C26 to C17, L4 to L1, R10 to R6, S1 to RESET, S2 to BOOT
Connections:
- new net INT1_ACCEL: IC1.INT1, U1.IO9
- new net INT1_GYRO: IC1.INT3, U1.IO11
- new net INT2_ACCEL: IC1.INT2, U1.IO10
- new net INT2_GYRO: IC1.INT4, U1.IO12
- new net N$10: M1.+, U2.OUT+
- new net N$11: M1.-, U2.OUT-
- new net N$12: D2.-, R8.2
- new net N$13: R8.1, U5.STAT
- new net N$15: R7.2, U5.PROG
- new net N$3: J5.+, Q1.D
- new net N$6: C9.1, U2.REG
- new net PDM_CLK: MK1.CLK, U1.IO47
- new net PDM_DATA: MK1.DATA, U1.IO48
- new net RTC_N: C3.2, R2.1, U1.IO16, Y1.1
- new net RTC_P: C2.2, R2.2, U1.IO15, Y1.2
- new net RX: J2.2, U1.RXD0
- new net SCL: IC1.SCX, J3.4, R3.1, U1.IO13, U2.SCL, U3.SCK
- new net SDA: IC1.SDX, J3.3, R4.1, U1.IO14, U2.SDA, U3.SDI
- new net TCK: J1.SWDCLK/TCK, U1.IO39
- new net TDI: J1.NC/TDI, U1.IO41
- new net TDO: J1.SWO/TDO, U1.IO40
- new net TMS: J1.SWDIO/TMS, U1.IO42
- new net TX: J2.3, U1.TXD0
- new net VIN: C14.2, D1.-, SW1.2, U4.EN, U4.VIN
- new net V_BATT: C18.2, Q1.S, SW1.1, U5.VBAT
- net 3.3V: now also C10.1, C11.1, C12.2, C13.2, C15.2, C20.1, C4.1, C5.1, C7.2, C8.1, IC1.PS, IC1.VDD, IC1.VDDIO, J1.VCC, J2.1, J3.2, MK1.VDD, R3.2, R4.2, U2.EN, U2.VDD, U2.VDD/NC, U3.CSB, U3.VDD, U3.VDDIO, U4.VOUT; no longer C2.1, C3.1
- net EN: now also C6.1, J1.!RESET; no longer C4.1
- net GND: now also C10.2, C11.2, C12.1, C13.1, C14.1, C15.1, C18.1, C19.1, C2.1, C20.2, C3.1, C5.2, C6.2, C7.1, C8.2, C9.2, IC1.GNDA, IC1.GNDIO, IC1.SDO1, IC1.SDO2, J1.GND@3, J1.GND@5, J1.GNDDTCT, J2.4, J2.SHIELD, J3.1, J4.GND, J5.-, MK1.GND, MK1.SELECT, R5.1, R7.1, SW1.SHIELD, U2.GND, U2.IN/TRIG, U3.GND, U3.SDO, U4.GND, U5.VSS, U6.GND; no longer C2.2, C3.2, J2.GND, U5.GND
- net N$1: now also J4.CC1, R5.2; no longer J2.CC1, R9.2
- net N$14: now also J4.VBUS; no longer J2.VBUS
- net N$2: now also J4.CC2; no longer J2.CC2
- net USBD_N: now also J4.DN1, J4.DN2, U6.I/O2_OUT; no longer J2.DN1, J2.DN2, U5.I/O2_OUT
- net USBD_P: now also J4.DP1, J4.DP2, U6.I/O1_OUT; no longer J2.DP1, J2.DP2, U5.I/O1_OUT
- net USB_N: now also U1.IO19, U6.I/O2_IN; no longer U5.I/O2_IN
- net USB_P: now also U1.IO20, U6.I/O1_IN; no longer U1.IO19, U5.I/O1_IN
- net V_USB: now also C19.2, D1.+, D2.+, Q1.G, R9.2, U5.VDD, U6.VBUS; no longer U5.VBUS
